File: pcb/valve.kicad_sch (KiCad schematic)
At the start: 6 parts, among them Q1 PMBT3904, Q2 SS8550-H

Commit message: Update resistor values based on availability
Parts:
- R1: value 4.3K -> 3.9K; CID 100.316.93 -> 100.014.54
Changed lines of the file:
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@@
 			)
 		)
-		(property "Value" "4.3K"
+		(property "Value" "3.9K"
 			(at 115.57 88.9 90)
 			(effects
@@
 			)
 		)
-		(property "CID" "100.316.93"
+		(property "CID" "100.014.54"
 			(at 115.57 92.71 90)
 			(effects

Commit message: Change terminal, add another output, add hardware debouncing
Connections:
- net +12V: now also Q2.2 (E); no longer Q2.3 (C)
- net OUT: now also Q2.3 (C); no longer Q2.2 (E)
Changed lines of the file:
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@@
+					(unit 1)
+				)
+				(path "/15d58363-062f-45fb-af18-cd9dd75f9ed5/f6855309-c20b-4afd-9ee1-6feb23f07aec"
+					(reference "D9")
 					(unit 1)
 				)
@@
 					(unit 1)
 				)
+				(path "/15d58363-062f-45fb-af18-cd9dd75f9ed5/f6855309-c20b-4afd-9ee1-6feb23f07aec"
+					(reference "Q9")
+					(unit 1)
+				)
 			)
 		)
@@
 					(unit 1)
 				)
+				(path "/15d58363-062f-45fb-af18-cd9dd75f9ed5/f6855309-c20b-4afd-9ee1-6feb23f07aec"
+					(reference "#PWR014")
+					(unit 1)
+				)
 			)
 		)
@@
 					(unit 1)
 				)
+				(path "/15d58363-062f-45fb-af18-cd9dd75f9ed5/f6855309-c20b-4afd-9ee1-6feb23f07aec"
+					(reference "#PWR015")
+					(unit 1)
+				)
 			)
 		)
@@
 		(lib_id "Device:Q_PNP_BEC")
 		(at 160.02 86.36 0)
+		(mirror x)
 		(unit 1)
 		(exclude_from_sim no)
@@
 		(fields_autoplaced yes)
 		(property "Reference" "Q2"
-			(at 165.1 85.0899 0)
+			(at 165.1 87.6301 0)
 			(effects
 				(font
@@
 		)
 		(property "Value" "SS8550-H"
-			(at 165.1 87.6299 0)
+			(at 165.1 85.0901 0)
 			(effects
 				(font
@@
 		)
 		(property "Footprint" "Package_TO_SOT_SMD:TSOT-23"
-			(at 165.1 83.82 0)
+			(at 165.1 88.9 0)
 			(effects
 				(font
@@
 				(path "/15d58363-062f-45fb-af18-cd9dd75f9ed5/f0d80cdd-41ca-4947-afbf-3715980c4b1b"
 					(reference "Q8")
+					(unit 1)
+				)
+				(path "/15d58363-062f-45fb-af18-cd9dd75f9ed5/f6855309-c20b-4afd-9ee1-6feb23f07aec"
+					(reference "Q10")
 					(unit 1)
 				)
@@
 					(unit 1)
 				)
+				(path "/15d58363-062f-45fb-af18-cd9dd75f9ed5/f6855309-c20b-4afd-9ee1-6feb23f07aec"
+					(reference "R10")
+					(unit 1)
+				)
 			)
 		)
@@
 					(unit 1)
 				)
+				(path "/15d58363-062f-45fb-af18-cd9dd75f9ed5/f6855309-c20b-4afd-9ee1-6feb23f07aec"
+					(reference "R9")
+					(unit 1)
+				)
 			)
 		)
@@
 					(unit 1)
 				)
+				(path "/15d58363-062f-45fb-af18-cd9dd75f9ed5/f6855309-c20b-4afd-9ee1-6feb23f07aec"
+					(reference "D10")
+					(unit 1)
+				)

Commit message: Adjust components based on availability
Parts:
- D1: value EVL-SMD0805-RED -> EVL-BHC-AN1P2; CID 100.432.15 -> 100.363.83
Changed lines of the file:
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@@
 			)
 		)
-		(property "Value" "EVL-SMD0805-RED"
+		(property "Value" "EVL-BHC-AN1P2"
 			(at 131.7625 81.28 0)
 			(effects
@@
 			)
 		)
-		(property "CID" "100.432.15"
+		(property "CID" "100.363.83"
 			(at 133.35 86.36 0)
 			(effects
